Commit message: Commit updated amr.urdf with frictionless front caster wheel

File: src/amr.urdf (robot description, URDF)
Before this commit: robot edge_amr, 6 links, 5 joints
Links:
- added link front_caster_link, mass 0.5; collision sphere radius=0.05; visual sphere radius=0.05
Joints:
- added joint front_caster_joint: type fixed, parent base_link, child front_caster_link, origin xyz=0.2 0 -0.15 rpy=0 0 0
